File: pcb/LCD_Matrix.kicad_sch (KiCad schematic)
At the start: 2 parts, among them J10 691137710003, J11 691137710003

Commit message: stuff
Parts:
- J10, J11: footprint 691137710003:691137710003 -> 3x1term:691137710003
Connections:
- no-connect marks 0 -> 1
Other:
- note added: "LED Matrix Connectors"
- moved on the sheet: J10, J11
Changed lines of the file:
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@@
 	(generator_version "9.0")
 	(paper "A4")
-	(wire
-		(pts
-			(xy 59.69 97.79) (xy 66.04 97.79)
-		)
-		(stroke
-			(width 0)
-			(type default)
-		)
-	)
-	(wire
-		(pts
-			(xy 72.39 73.66) (xy 72.39 74.93)
-		)
-		(stroke
-			(width 0)
-			(type default)
-		)
-	)
-	(wire
-		(pts
-			(xy 59.69 92.71) (xy 66.04 92.71)
-		)
-		(stroke
-			(width 0)
-			(type default)
-		)
-	)
-	(wire
-		(pts
-			(xy 66.04 97.79) (xy 66.04 99.06)
-		)
-		(stroke
-			(width 0)
-			(type default)
-		)
-	)
-	(wire
-		(pts
-			(xy 59.69 76.2) (xy 68.58 76.2)
-		)
-		(stroke
-			(width 0)
-			(type default)
-		)
-	)
-	(wire
-		(pts
-			(xy 59.69 73.66) (xy 72.39 73.66)
-		)
-		(stroke
-			(width 0)
-			(type default)
-		)
-	)
-	(wire
-		(pts
-			(xy 59.69 71.12) (xy 66.04 71.12)
-		)
-		(stroke
-			(width 0)
-			(type default)
-		)
-	)
-	(label "LED_Data"
-		(at 68.58 76.2 180)
+	(rectangle
+		(start 113.03 74.93)
+		(end 185.42 109.22)
+		(stroke
+			(width 0)
+			(type default)
+		)
+		(fill
+			(type none)
+		)
+	)
+	(text "LED Matrix Connectors"
+		(exclude_from_sim no)
+		(at 147.828 80.772 0)
 		(effects
 			(font
 				(size 1.27 1.27)
 			)
-			(justify right bottom)
+		)
+	)
+	(no_connect
+		(at 170.18 96.52)
+	)
+	(wire
+		(pts
+			(xy 170.18 99.06) (xy 176.53 99.06)
+		)
+		(stroke
+			(width 0)
+			(type default)
+		)
+	)
+	(wire
+		(pts
+			(xy 143.51 96.52) (xy 143.51 97.79)
+		)
+		(stroke
+			(width 0)
+			(type default)
+		)
+	)
+	(wire
+		(pts
+			(xy 170.18 93.98) (xy 176.53 93.98)
+		)
+		(stroke
+			(width 0)
+			(type default)
+		)
+	)
+	(wire
+		(pts
+			(xy 176.53 99.06) (xy 176.53 100.33)
+		)
+		(stroke
+			(width 0)
+			(type default)
+		)
+	)
+	(wire
+		(pts
+			(xy 125.73 99.06) (xy 129.54 99.06)
+		)
+		(stroke
+			(width 0)
+			(type default)
+		)
+	)
+	(wire
+		(pts
+			(xy 125.73 96.52) (xy 143.51 96.52)
+		)
+		(stroke
+			(width 0)
+			(type default)
+		)
+	)
+	(wire
+		(pts
+			(xy 125.73 93.98) (xy 132.08 93.98)
+		)
+		(stroke
+			(width 0)
+			(type default)
+		)
+	)
+	(hierarchical_label "LED_Data"
+		(shape input)
+		(at 129.54 99.06 0)
+		(effects
+			(font
+				(size 1.27 1.27)
+			)
+			(justify left)
 		)
 	)
 	(symbol
 		(lib_id "screw_terminal:691137710003")
-		(at 54.61 73.66 90)
+		(at 120.65 96.52 90)
 		(unit 1)
 		(exclude_from_sim no)
@@
 		(fields_autoplaced yes)
 		(property "Reference" "J10"
-			(at 55.88 64.77 90)
+			(at 121.92 87.63 90)
 			(effects
 				(font
@@
 		)
 		(property "Value" "691137710003"
-			(at 55.88 67.31 90)
-			(effects
-				(font
-					(size 1.27 1.27)
-				)
-			)
-		)
-		(property "Footprint" "691137710003:691137710003"
-			(at 54.61 73.66 0)
+			(at 121.92 90.17 90)
+			(effects
+				(font
+					(size 1.27 1.27)
+				)
+			)
+		)
+		(property "Footprint" "3x1term:691137710003"
+			(at 120.65 96.52 0)
 			(effects
 				(font
@@
 		)
 		(property "Datasheet" ""
-			(at 54.61 73.66 0)
+			(at 120.65 96.52 0)
 			(effects
 				(font
@@
 		)
 		(property "Description" ""
-			(at 54.61 73.66 0)
+			(at 120.65 96.52 0)
 			(effects
 				(font
@@
 	(symbol
 		(lib_id "power:+5V")
-		(at 66.04 92.71 0)
+		(at 176.53 93.98 0)
 		(unit 1)
 		(exclude_from_sim no)
@@
 		(fields_autoplaced yes)
 		(property "Reference" "#PWR042"
-			(at 66.04 96.52 0)
+			(at 176.53 97.79 0)
 			(effects
 				(font
@@
 		)
 		(property "Value" "+5V"
-			(at 66.04 87.63 0)
+			(at 176.53 88.9 0)
 			(effects
 				(font
@@
 		)
 		(property "Footprint" ""
-			(at 66.04 92.71 0)
-			(effects
-				(font
-					(size 1.27 1.27)
-				)
-				(hide yes)
-			)
-		)
-		(property "Datasheet" ""
-			(at 66.04 92.71 0)
+			(at 176.53 93.98 0)
+			(effects
+				(font
+					(size 1.27 1.27)
+				)
+				(hide yes)
+			)
+		)
+		(property "Datasheet" ""
+			(at 176.53 93.98 0)
 			(effects
 				(font
@@
 		)
 		(property "Description" "Power symbol creates a global label with name \"+5V\""
-			(at 66.04 92.71 0)
+			(at 176.53 93.98 0)
 			(effects
 				(font
@@
 	(symbol
 		(lib_id "screw_terminal:691137710003")
-		(at 54.61 95.25 90)
+		(at 165.1 96.52 90)
 		(unit 1)
 		(exclude_from_sim no)
@@
 		(fields_autoplaced yes)
 		(property "Reference" "J11"
-			(at 55.88 86.36 90)
+			(at 166.37 87.63 90)
 			(effects
 				(font
@@
 		)
 		(property "Value" "691137710003"
-			(at 55.88 88.9 90)
-			(effects
-				(font
-					(size 1.27 1.27)
-				)
-			)
-		)
-		(property "Footprint" "691137710003:691137710003"
-			(at 54.61 95.25 0)
+			(at 166.37 90.17 90)
+			(effects
+				(font
+					(size 1.27 1.27)
+				)
+			)
+		)
+		(property "Footprint" "3x1term:691137710003"
+			(at 165.1 96.52 0)
 			(effects
 				(font
@@
 		)
 		(property "Datasheet" ""
-			(at 54.61 95.25 0)
+			(at 165.1 96.52 0)
 			(effects
 				(font
@@
 		)
 		(property "Description" ""
-			(at 54.61 95.25 0)
+			(at 165.1 96.52 0)
 			(effects
 				(font
@@
 	(symbol
 		(lib_id "power:GND")
-		(at 72.39 74.93 0)
+		(at 143.51 97.79 0)
 		(unit 1)
 		(exclude_from_sim no)
@@
 		(fields_autoplaced yes)
 		(property "Reference" "#PWR041"
-			(at 72.39 81.28 0)
+			(at 143.51 104.14 0)
 			(effects
 				(font
@@
 		)
 		(property "Value" "GND"
-			(at 72.39 80.01 0)
+			(at 143.51 102.87 0)
 			(effects
 				(font
@@
 		)
 		(property "Footprint" ""
-			(at 72.39 74.93 0)
-			(effects
-				(font
-					(size 1.27 1.27)
-				)
-				(hide yes)
-			)
-		)
-		(property "Datasheet" ""
-			(at 72.39 74.93 0)
+			(at 143.51 97.79 0)
+			(effects
+				(font
+					(size 1.27 1.27)
+				)
+				(hide yes)
+			)
+		)
+		(property "Datasheet" ""
+			(at 143.51 97.79 0)
 			(effects
 				(font
@@
 		)
 		(property "Description" "Power symbol creates a global label with name \"GND\" , ground"
-			(at 72.39 74.93 0)
+			(at 143.51 97.79 0)
 			(effects
 				(font
@@
 	(symbol
 		(lib_id "power:+5V")
-		(at 66.04 71.12 0)
+		(at 132.08 93.98 0)
 		(unit 1)
 		(exclude_from_sim no)
@@
 		(fields_autoplaced yes)
 		(property "Reference" "#PWR040"
-			(at 66.04 74.93 0)
+			(at 132.08 97.79 0)
 			(effects
 				(font
@@
 		)
 		(property "Value" "+5V"
-			(at 66.04 66.04 0)
+			(at 132.08 88.9 0)
 			(effects
 				(font
@@
 		)
 		(property "Footprint" ""
-			(at 66.04 71.12 0)
-			(effects
-				(font
-					(size 1.27 1.27)
-				)
-				(hide yes)
-			)
-		)
-		(property "Datasheet" ""
-			(at 66.04 71.12 0)
+			(at 132.08 93.98 0)
+			(effects
+				(font
+					(size 1.27 1.27)
+				)
+				(hide yes)
+			)
+		)
+		(property "Datasheet" ""
+			(at 132.08 93.98 0)
 			(effects
 				(font
@@
 		)
 		(property "Description" "Power symbol creates a global label with name \"+5V\""
-			(at 66.04 71.12 0)
+			(at 132.08 93.98 0)
 			(effects
 				(font
@@
 	(symbol
 		(lib_id "power:GND")
-		(at 66.04 99.06 0)
+		(at 176.53 100.33 0)
 		(unit 1)
 		(exclude_from_sim no)
@@
 		(fields_autoplaced yes)
 		(property "Reference" "#PWR043"
-			(at 66.04 105.41 0)
+			(at 176.53 106.68 0)
 			(effects
 				(font
@@
 		)
 		(property "Value" "GND"
-			(at 66.04 104.14 0)
+			(at 176.53 105.41 0)
 			(effects
 				(font
@@
 		)
 		(property "Footprint" ""
-			(at 66.04 99.06 0)
-			(effects
-				(font
-					(size 1.27 1.27)
-				)
-				(hide yes)
-			)
-		)
-		(property "Datasheet" ""
-			(at 66.04 99.06 0)
+			(at 176.53 100.33 0)
+			(effects
+				(font
+					(size 1.27 1.27)
+				)
+				(hide yes)
+			)
+		)
+		(property "Datasheet" ""
+			(at 176.53 100.33 0)
 			(effects
 				(font
@@
 		)
 		(property "Description" "Power symbol creates a global label with name \"GND\" , ground"
-			(at 66.04 99.06 0)
-			(effects
-				(font
+			(at 176.53 100.33 0)
+			(effects
+				(font
