File: pcb/power.kicad_sch (KiCad schematic)
At the start: 5 parts, among them J1 73099-0, J12 73099-0, U4 AZ1117IH-3.3TRG1

Commit message: stuff
Parts:
- removed J1, J12: 73099-0, 73099-0:POMONA_73099-0, symbol banana_plug:73099-0
- added D1, D3: LED, symbol Device:LED
- added P1: USB_C_Plug_USB2.0, symbol Connector:USB_C_Plug_USB2.0
- added R1, R8: 5.1K, symbol Device:R
- added R10, R9: 220, symbol Device:R
- added TP7, TP8: TestPoint, symbol Connector:TestPoint
Connections:
- net +3.3V: now also R10.2
- net +5V: now also P1.A4 (VBUS), P1.A9 (VBUS), P1.B4 (VBUS), P1.B9 (VBUS), R9.2, TP7.1
- net GND: now also D1.1 (K), D3.1 (K), P1.A1 (GND), P1.A12 (GND), P1.B1 (GND), P1.B12 (GND), P1.S1 (SHIELD), R1.2, R8.1, TP8.1
- new net: D1.2 (A), R9.1
- new net: D3.2 (A), R10.1
- new net: P1.A5 (CC), R1.1
- new net: P1.B5 (VCONN), R8.2
- no-connect marks 0 -> 2
Other:
- note added: "not plug"
- moved on the sheet: TP5, TP6

Commit message: stuff
Parts:
- removed P1: USB_C_Plug_USB2.0, symbol Connector:USB_C_Plug_USB2.0
- added C1: 10uF, Capacitor_SMD:C_0603_1608Metric, symbol Device:C_Polarized
- added C2: 22uF, Capacitor_SMD:C_0603_1608Metric, symbol Device:C_Polarized
- added J15: USB_C_Receptacle_PowerOnly_6P, Connector_USB:USB_C_Receptacle_GCT_USB4125-xx-x-0190_6P_TopMnt_Horizontal, symbol Connector:USB_C_Receptacle_PowerOnly_6P
- added TP10, TP9: TestPoint, TestPoint:TestPoint_Pad_3.0x3.0mm, symbol Connector:TestPoint
- D1, D3: footprint (none) -> LED_SMD:LED_0603_1608Metric
- R1, R10, R8, R9: footprint (none) -> Resistor_SMD:R_0603_1608Metric
- TP5, TP6, TP7, TP8: footprint (none) -> TestPoint:TestPoint_Pad_3.0x3.0mm
- U4: footprint AZ1117IH-3.3TRG1:SOT230P700X185-4N -> ldo:SOT230P700X185-4N
Connections:
- net +3.3V: now also C2.1, TP9.1
- net +5V: now also C1.1, J15.A9 (VBUS), J15.B9 (VBUS)
- net GND: now also C1.2, C2.2, J15.A12 (GND), J15.B12 (GND), J15.S1 (SHIELD), TP10.1
- net at R1.1: now also J15.A5 (CC1)
- net at R8.2: now also J15.B5 (CC2)
- no-connect marks 2 -> 0
Other:
- note added: "LDO from 5V to 3.3V Used for IC power"
- note added: "Power and GND Testpoints / Power Leds"
- note added: "USB-C Power Delivery 5.1k resistors tied to CC lines for 5v @ 3A"
- note removed: "not plug"
- moved on the sheet: D1, D3, R1, R10, R8, R9, TP5, TP6, TP7, TP8, U4
