File: pcb/receiver.kicad_sch (KiCad schematic)
At the start: 1 part, among them J2 Conn_01x05_Socket

Commit message: stuff
Other:
- note added: "IR Receiver Breakout Board Connector"
- moved on the sheet: J2
Changed lines of the file:
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@@
 	(generator_version "9.0")
 	(paper "A4")
-	(wire
-		(pts
-			(xy 147.32 113.03) (xy 154.94 113.03)
-		)
-		(stroke
-			(width 0)
-			(type default)
-		)
-	)
-	(wire
-		(pts
-			(xy 147.32 120.65) (xy 154.94 120.65)
-		)
-		(stroke
-			(width 0)
-			(type default)
-		)
-	)
-	(wire
-		(pts
-			(xy 163.83 116.84) (xy 163.83 118.11)
-		)
-		(stroke
-			(width 0)
-			(type default)
-		)
-	)
-	(wire
-		(pts
-			(xy 147.32 118.11) (xy 163.83 118.11)
-		)
-		(stroke
-			(width 0)
-			(type default)
-		)
-	)
-	(wire
-		(pts
-			(xy 147.32 115.57) (xy 154.94 115.57)
-		)
-		(stroke
-			(width 0)
-			(type default)
-		)
-	)
-	(wire
-		(pts
-			(xy 147.32 110.49) (xy 154.94 110.49)
-		)
-		(stroke
-			(width 0)
-			(type default)
-		)
-	)
-	(label "IRH"
-		(at 154.94 110.49 0)
-		(effects
-			(font
-				(size 1.27 1.27)
-			)
-			(justify left bottom)
-		)
-	)
-	(label "Sig"
-		(at 154.94 115.57 0)
-		(effects
-			(font
-				(size 1.27 1.27)
-			)
-			(justify left bottom)
-		)
-	)
-	(label "IRV"
-		(at 154.94 113.03 0)
-		(effects
-			(font
-				(size 1.27 1.27)
-			)
-			(justify left bottom)
+	(rectangle
+		(start 107.95 82.55)
+		(end 175.26 121.92)
+		(stroke
+			(width 0)
+			(type default)
+		)
+		(fill
+			(type none)
+		)
+	)
+	(text "IR Receiver Breakout Board Connector\n\n"
+		(exclude_from_sim no)
+		(at 143.002 88.392 0)
+		(effects
+			(font
+				(size 1.27 1.27)
+			)
+		)
+	)
+	(wire
+		(pts
+			(xy 140.97 104.14) (xy 149.86 104.14)
+		)
+		(stroke
+			(width 0)
+			(type default)
+		)
+	)
+	(wire
+		(pts
+			(xy 140.97 111.76) (xy 148.59 111.76)
+		)
+		(stroke
+			(width 0)
+			(type default)
+		)
+	)
+	(wire
+		(pts
+			(xy 161.29 107.95) (xy 161.29 109.22)
+		)
+		(stroke
+			(width 0)
+			(type default)
+		)
+	)
+	(wire
+		(pts
+			(xy 140.97 109.22) (xy 161.29 109.22)
+		)
+		(stroke
+			(width 0)
+			(type default)
+		)
+	)
+	(wire
+		(pts
+			(xy 140.97 106.68) (xy 149.86 106.68)
+		)
+		(stroke
+			(width 0)
+			(type default)
+		)
+	)
+	(wire
+		(pts
+			(xy 140.97 101.6) (xy 149.86 101.6)
+		)
+		(stroke
+			(width 0)
+			(type default)
+		)
+	)
+	(hierarchical_label "Sig"
+		(shape input)
+		(at 149.86 106.68 0)
+		(effects
+			(font
+				(size 1.27 1.27)
+			)
+			(justify left)
+		)
+	)
+	(hierarchical_label "IRV"
+		(shape input)
+		(at 149.86 104.14 0)
+		(effects
+			(font
+				(size 1.27 1.27)
+			)
+			(justify left)
+		)
+	)
+	(hierarchical_label "IRH"
+		(shape input)
+		(at 149.86 101.6 0)
+		(effects
+			(font
+				(size 1.27 1.27)
+			)
+			(justify left)
 		)
 	)
 	(symbol
 		(lib_id "power:GND")
-		(at 154.94 120.65 0)
+		(at 148.59 111.76 0)
 		(unit 1)
 		(exclude_from_sim no)
@@
 		(fields_autoplaced yes)
 		(property "Reference" "#PWR02"
-			(at 154.94 127 0)
+			(at 148.59 118.11 0)
 			(effects
 				(font
@@
 		)
 		(property "Value" "GND"
-			(at 154.94 125.73 0)
+			(at 148.59 116.84 0)
 			(effects
 				(font
@@
 		)
 		(property "Footprint" ""
-			(at 154.94 120.65 0)
+			(at 148.59 111.76 0)
 			(effects
 				(font
@@
 		)
 		(property "Datasheet" ""
-			(at 154.94 120.65 0)
+			(at 148.59 111.76 0)
 			(effects
 				(font
@@
 		)
 		(property "Description" "Power symbol creates a global label with name \"GND\" , ground"
-			(at 154.94 120.65 0)
+			(at 148.59 111.76 0)
 			(effects
 				(font
@@
 	(symbol
 		(lib_id "Connector:Conn_01x05_Socket")
-		(at 142.24 115.57 180)
+		(at 135.89 106.68 180)
 		(unit 1)
 		(exclude_from_sim no)
@@
 		(fields_autoplaced yes)
 		(property "Reference" "J2"
-			(at 142.875 105.41 0)
+			(at 136.525 96.52 0)
 			(effects
 				(font
@@
 		)
 		(property "Value" "Conn_01x05_Socket"
-			(at 142.875 107.95 0)
+			(at 136.525 99.06 0)
 			(effects
 				(font
@@
 		)
 		(property "Footprint" "Connector_PinHeader_2.54mm:PinHeader_1x05_P2.54mm_Vertical"
-			(at 142.24 115.57 0)
+			(at 135.89 106.68 0)
 			(effects
 				(font
@@
 		)
 		(property "Datasheet" "~"
-			(at 142.24 115.57 0)
+			(at 135.89 106.68 0)
 			(effects
 				(font
@@
 		)
 		(property "Description" "Generic connector, single row, 01x05, script generated"
-			(at 142.24 115.57 0)
+			(at 135.89 106.68 0)
 			(effects
 				(font
@@
 	(symbol
 		(lib_id "power:+3.3V")
-		(at 163.83 116.84 0)
+		(at 161.29 107.95 0)
 		(unit 1)
 		(exclude_from_sim no)
@@
 		(fields_autoplaced yes)
 		(property "Reference" "#PWR01"
-			(at 163.83 120.65 0)
+			(at 161.29 111.76 0)
 			(effects
 				(font
@@
 		)
 		(property "Value" "+3.3V"
-			(at 163.83 111.76 0)
+			(at 161.29 102.87 0)
 			(effects
 				(font
@@
 		)
 		(property "Footprint" ""
-			(at 163.83 116.84 0)
+			(at 161.29 107.95 0)
 			(effects
 				(font
@@
 		)
 		(property "Datasheet" ""
-			(at 163.83 116.84 0)
+			(at 161.29 107.95 0)
 			(effects
 				(font
@@
 		)
 		(property "Description" "Power symbol creates a global label with name \"+3.3V\""
-			(at 163.83 116.84 0)
-			(effects
-				(font
+			(at 161.29 107.95 0)
+			(effects
+				(font
