File: pcb/IMU.kicad_sch (KiCad schematic)
At the start: 2 parts, among them J9 284414-6, U2 4754

Commit message: stuff
Parts:
- J9: footprint CONN6_284414-6_TEC -> 6x1term:CONN6_284414-6_TEC
- U2: footprint 4754:MODULE_4754 -> bno085:MODULE_4754
Connections:
- no-connect marks 2 -> 6
Other:
- note added: "BNO085 Breakout Board Connector"
- note added: "Wand IMU Screw Terminal"
- moved on the sheet: J9, U2

Commit message: board
Connections:
- net INT_IMU: now also J9.3; no longer J9.2
- net RST_IMU: now also J9.2; no longer J9.3
Changed lines of the file:
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@@
-		)
-	)
-	(label "RST_IMU"
-		(at 73.66 118.11 180)
-		(effects
-			(font
-				(size 1.27 1.27)
-			)
-			(justify right bottom)
 		)
 	)
@@
 		)
 	)
-	(label "INT_IMU"
+	(label "RST_IMU"
 		(at 73.66 120.65 180)
 		(effects
 			(font
+				(size 1.27 1.27)
+			)
+			(justify right bottom)
+		)
+	)
+	(label "INT_IMU"
+		(at 73.66 118.11 180)
+		(effects
+			(font
