File: pcb/emitter.kicad_sch (KiCad schematic)
At the start: 16 parts, among them J3 1751248, J4 1751248, J5 Conn_01x03_Pin, J6 Conn_01x03_Pin, Q1 AO3406

Commit message: stuff
Parts:
- removed C4: 10uF, symbol Device:C
- removed J5, J6: Conn_01x03_Pin, Connector_PinHeader_2.54mm:PinHeader_1x03_P2.54mm_Vertical, symbol Connector:Conn_01x03_Pin
- removed JP4: Jumper_2_Open, TestPoint:TestPoint_2Pads_Pitch5.08mm_Drill1.3mm, symbol Jumper:Jumper_2_Open
- added J5: Conn_01x03_Socket, Connector_PinSocket_2.54mm:PinSocket_1x03_P2.54mm_Vertical, symbol Connector:Conn_01x03_Socket
- C5, C6, C7: footprint (none) -> Capacitor_SMD:C_0603_1608Metric
- D2: footprint (none) -> LED_SMD:LED_0603_1608Metric
- J3, J4: footprint CONN_1751248_PXC -> 2x1term:CONN_1751248_PXC
- JP3: footprint TestPoint:TestPoint_2Pads_Pitch5.08mm_Drill1.3mm -> TestPoint:TestPoint_2Pads_Pitch2.54mm_Drill0.8mm
- R2, R3, R4, R5: footprint (none) -> Resistor_SMD:R_0603_1608Metric
Connections:
- net +3.3V: now also J5.2 (Pin_2)
- net GND: now also J5.1 (Pin_1)
- net emitter_out: now also J5.3 (Pin_3)
Other:
- note added: "IR Breakout Board Connector"
- note added: "LED Circuitry"
- note added: "Screw Terminal To Wand For IR LEDs"
- moved on the sheet: C5, C6, C7, D2, J3, J4, JP3, Q1, R2, R3, R4, R5

Commit message: board
Parts:
- Q1: footprint IR STEMMA LED Emitter:SOT23-WIDE -> Package_TO_SOT_SMD:SOT-23-3
Changed lines of the file:
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@@
 			)
 		)
-		(property "Footprint" "IR STEMMA LED Emitter:SOT23-WIDE"
+		(property "Footprint" "Package_TO_SOT_SMD:SOT-23-3"
 			(at 85.09 140.97 0)
 			(effects
