File: pcb/proton.kicad_sch (KiCad schematic)
At the start: 0 parts

Commit message: stuff
Parts:
- added J1, J12: Conn_01x28_Socket, Connector_PinSocket_2.54mm:PinSocket_1x28_P2.54mm_Vertical, symbol Connector:Conn_01x28_Socket
- added J13: Conn_01x04_Socket, Connector_PinHeader_2.54mm:PinHeader_1x04_P2.54mm_Vertical, symbol Connector:Conn_01x04_Socket
- added J14: Conn_01x03_Socket, symbol Connector:Conn_01x03_Socket
Other:
- note added: "17.78mm between sides 15.24mm from GND to Probe USB BOOT"

Commit message: stuff
Parts:
- added J6: 691137710003, 3x1term:691137710003, symbol screw_terminal:691137710003
- J14: footprint (none) -> Connector_PinSocket_2.54mm:PinSocket_1x01_P2.54mm_Vertical
Connections:
- net +5V: now reaches J12.1 (Pin_1)
- net +5V: now also J1.1 (Pin_1)
- net SWCLK: now reaches J12.26 (Pin_26)
- net SWCLK: now also J13.2 (Pin_2)
- net SWD: now reaches J12.27 (Pin_27)
- net SWD: now also J13.4 (Pin_4)
- net GND: now reaches J12.28 (Pin_28)
- net GND: now also J1.28 (Pin_28), J13.3 (Pin_3), J14.2 (Pin_2)
- net IRV: now reaches J1.10 (Pin_10)
- net IRH: now reaches J1.11 (Pin_11)
- net RST_IMU: now reaches J1.12 (Pin_12)
- net INT_IMU: now reaches J1.13 (Pin_13)
- net Button1: now reaches J1.16 (Pin_16)
- net Button1: now also J6.3
- net Button2: now reaches J1.17 (Pin_17)
- net Button2: now also J6.2
- net Button3: now reaches J1.18 (Pin_18)
- net Button3: now also J6.1
- net emitter_out: now reaches J1.19 (Pin_19)
- net haptics_trig1: now reaches J1.21 (Pin_21)
- net haptics_trig2: now reaches J1.22 (Pin_22)
- net LED_Data: now reaches J1.23 (Pin_23)
- net Proton_RX: now reaches J1.3 (Pin_3)
- net Proton_RX: now also J14.3 (Pin_3)
- net Proton_TX: now reaches J1.4 (Pin_4)
- net Proton_TX: now also J14.1 (Pin_1)
- net SDA2: now reaches J1.5 (Pin_5)
- net SCL2: now reaches J1.6 (Pin_6)
- net SDA1: now reaches J1.7 (Pin_7)
- net SCL1: now reaches J1.8 (Pin_8)
- net Sig: now reaches J1.9 (Pin_9)
- no-connect marks 0 -> 33
Other:
- note added: "GPIO 10 / IMU Interrupt"
- note added: "GPIO 13 / Wand Button 1"
- note added: "GPIO 14 / Wand Button 2"
- note added: "GPIO 15 / Wand Button 3"
- note added: "GPIO 16 / PWM0 A / IR Emitter"
- note added: "GPIO 18 / PWM1 A / Haptics 1"
- note added: "GPIO 19 / PWM1 B / Haptics 2"
- note added: "GPIO 2 / I2C1 SDA / Haptics 2"
- note added: "GPIO 20 / LED Data In"
- note added: "GPIO 3 / I2C1 SCL / Haptics 2"
- note added: "GPIO 4 / I2C0 SDA"
- note added: "GPIO 5 / I2C0 SCL"
- note added: "GPIO 6 / Reciever Signal"
- note added: "GPIO 7 / Reciever Signal Vertical"
- note added: "GPIO 8 / Reciever Signal Horizantal"
- note added: "GPIO 9 / IMU Reset"
- moved on the sheet: J12, J13, J14

Commit message: board
Parts:
- added J16, J18: Conn_01x28_Socket, Connector_PinSocket_2.54mm:PinSocket_1x28_P2.54mm_Vertical, symbol Connector:Conn_01x28_Socket
- added J17: Conn_01x03_Socket, Connector_PinSocket_2.54mm:PinSocket_1x03_P2.54mm_Vertical, symbol Connector:Conn_01x03_Socket
- added J19: Conn_01x04_Socket, Connector_PinHeader_2.54mm:PinHeader_1x04_P2.54mm_Vertical, symbol Connector:Conn_01x04_Socket
- added JP4, JP5, JP6, JP7, JP8, JP9: Jumper_2_Open, TestPoint:TestPoint_2Pads_Pitch2.54mm_Drill0.8mm, symbol Jumper:Jumper_2_Open
- J14: footprint Connector_PinSocket_2.54mm:PinSocket_1x01_P2.54mm_Vertical -> Connector_PinSocket_2.54mm:PinSocket_1x03_P2.54mm_Vertical
Connections:
- net +5V: now also J16.1 (Pin_1), J18.1 (Pin_1)
- net GND: now also J16.28 (Pin_28), J17.2 (Pin_2), J18.28 (Pin_28), J19.3 (Pin_3)
- net INT_IMU: now also JP9.2 (B)
- net RST_IMU: now also JP8.1 (A)
- net SCL1: now also JP6.2 (B)
- net SCL2: now also JP5.2 (B)
- net SDA1: now also JP7.1 (A)
- net SDA2: now also JP4.1 (A)
- net SPI_RX: now reaches J12.22 (Pin_22)
- net SPI_RX: now also J18.22 (Pin_22)
- net SPI_TX: now reaches J12.23 (Pin_23)
- net SPI_TX: now also J18.23 (Pin_23)
- net SPI_CLK: now reaches J12.24 (Pin_24)
- net SPI_CLK: now also J18.24 (Pin_24)
- net SPI_CS: now reaches J12.25 (Pin_25)
- net SPI_CS: now also J18.25 (Pin_25)
- new net: J16.6 (Pin_6), JP5.1 (A)
- new net: J16.8 (Pin_8), JP6.1 (A)
- new net: J16.7 (Pin_7), JP7.2 (B)
- new net: J16.12 (Pin_12), JP8.2 (B)
- new net: J16.13 (Pin_13), JP9.1 (A)
- new net: J16.5 (Pin_5), JP4.2 (B)
- new net Proton_RX1: J16.3 (Pin_3), J17.3 (Pin_3)
- new net Proton_TX1: J16.4 (Pin_4), J17.1 (Pin_1)
- new net SWCLK1: J18.26 (Pin_26), J19.2 (Pin_2)
- new net SWD1: J18.27 (Pin_27), J19.4 (Pin_4)
- no-connect marks 33 -> 68
Other:
- note added: "Backup Wand Buttons"
- moved on the sheet: J1, J12, J13, J14, J6
