File: pcb/ece362project.kicad_pcb (KiCad board)
At the start: 2 copper layers, 160 x 160 mm, 67 parts, among them J1 Conn_01x28_Socket, J10 691137710003, J11 691137710003, J12 Conn_01x28_Socket, J13 Conn_01x04_Socket, J14 Conn_01x03_Socket, J15 USB_C_Receptacle_PowerOnly_6P, J16 Conn_01x28_Socket, J17 Conn_01x03_Socket, J18 Conn_01x28_Socket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

Commit message: stuff
Other:
- board text added: "INT"
- board text added: "RST"
- board text added: "SCL"
- board text added: "SDA"
Changed lines of the file:
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@@
+		)
+	)
+	(gr_text "GND"
+		(at 34.025 110.475 0)
+		(layer "F.SilkS")
+		(effects
+			(font
+				(size 1 1)
+				(thickness 0.1)
+			)
+			(justify left bottom)
 		)
 	)
@@
 		)
 	)
+	(gr_text "SCL"
+		(at 34.025 124.25 0)
+		(layer "F.SilkS")
+		(effects
+			(font
+				(size 1 1)
+				(thickness 0.1)
+			)
+			(justify left bottom)
+		)
+	)
 	(gr_text "Button 3"
 		(at 29.9 146.85 0)
@@
 		)
 	)
+	(gr_text "PWR"
+		(at 34.15 127.675 0)
+		(layer "F.SilkS")
+		(effects
+			(font
+				(size 1 1)
+				(thickness 0.1)
+			)
+			(justify left bottom)
+		)
+	)
 	(gr_text "3.3V\n"
 		(at 18.25 75.8 0)
@@
 		)
 	)
+	(gr_text "INT"
+		(at 34.2 117.25 0)
+		(layer "F.SilkS")
+		(effects
+			(font
+				(size 1 1)
+				(thickness 0.1)
+			)
+			(justify left bottom)
+		)
+	)
 	(gr_text "LED GND"
 		(at 23.25 176.4 0)
@@
 		(layer "F.SilkS")
 		(effects
+			(font
+				(size 1 1)
+				(thickness 0.1)
+			)
+			(justify left bottom)
+		)
+	)
+	(gr_text "SDA"
+		(at 34.1 120.8 0)
+		(layer "F.SilkS")
+		(effects
+			(font
+				(size 1 1)
+				(thickness 0.1)
+			)
+			(justify left bottom)
+		)
+	)
+	(gr_text "RST"
+		(at 34.1 113.875 0)
+		(layer "F.SilkS")
+		(effects
