File: pcb/ece362project.kicad_sch (KiCad schematic)
At the start: 0 parts

Commit message: stuff
Other:
- sheet IMU ports: added INT_IMU, RST_IMU, SCL1, SDA1; removed none
- sheet LCD_Matrix ports: added LED_Data; removed none
- sheet emitter ports: added emitter_out; removed none
- sheet haptics ports: added SCL1, SCL2, SDA1, SDA2, haptics_trig1, haptics_trig2; removed none
- sheet proton ports: added INT_IMU, IRH, IRV, LED_Data, RST_IMU, SCL1, SCL2, SDA1, SDA2, Sig, emitter_out, haptics_trig1, haptics_trig2; removed none
- sheet receiver ports: added IRH, IRV, Sig; removed none
- note added: "BNO085 IMU https://www.adafruit.com/product/4754 Used for gesture recognition to cast spells. Placed in the wand"
- note added: "Haptics Controllers https://www.adafruit.com/product/2305 Haptic motor controllers. The motors are in the wand, connected through the screw terminals. Non - Addressable I2C so split between two lines Used for user effects on the wand."
- note added: "IR Emitter https://learn.adafruit.com/adafruit-high-power-infrared-led-emitter Used for transmitting hit affect to target. PWM from proton."
- note added: "IR Receiver https://www.adafruit.com/product/5939 Receives 38Khz. Used for receiving led hit effect from opponent. GPIO to Proton."
- note added: "LED Matrix BTF-Lighting WS2812B LED Matrix used for displaying effects such as hits and health"
- note added: "Power Delivery 5v USB-C Input. 5v - 3.3v LDO. LDO 3.3v out used for logic power. Power Testpoints and Indicator LEDS."

Commit message: board
Other:
- title: (none) -> Chestplate PCB
Changed lines of the file:
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@@
 	(generator_version "9.0")
 	(paper "A4")
+	(title_block
+		(title "Chestplate PCB")
+	)
 	(text "IR Emitter \nhttps://learn.adafruit.com/adafruit-high-power-infrared-led-emitter\nUsed for transmitting hit affect to target. \nPWM from proton."
 		(exclude_from_sim no)
